File: eagle/usbdmx/usbdmx.brd (EAGLE design)
At the start: 63.2 x 48.6 mm, 35 parts, among them IC1 MAX3468CSA, IC2 MAX3468CSA, Q1 16MHz

Commit message: fix the polarity mixup on the secondary side
Parts:
- moved LED1 2.88 mm to (18.4, 13.3)
- moved R4 1.85 mm to (14.6, 12.7), turned to 0 degrees
- turned C8 to 180 degrees
Connections:
- net SGND: now also C8.1, U$2.7; no longer C8.2, U$2.8
- net SVCC: now also C8.2, U$2.8; no longer C8.1, U$2.7
Routing:
- net SVCC: track 55.1 -> 52.9 mm
- net SGND: track 132.0 -> 132.6 mm
Changed lines of the file:
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@@
 <grid distance="0.0125" unitdist="inch" unit="inch" style="lines" multiple="1" display="no" altdistance="0.025" altunitdist="inch" altunit="inch"/>
 <layers>
-<layer number="1" name="Top" color="4" fill="1" visible="no" active="yes"/>
+<layer number="1" name="Top" color="4" fill="1" visible="yes" active="yes"/>
 <layer number="16" name="Bottom" color="1" fill="1" visible="yes" active="yes"/>
 <layer number="17" name="Pads" color="2" fill="1" visible="yes" active="yes"/>
@@
 <layer number="23" name="tOrigins" color="15" fill="1" visible="yes" active="yes"/>
 <layer number="24" name="bOrigins" color="15" fill="1" visible="yes" active="yes"/>
-<layer number="25" name="tNames" color="7" fill="1" visible="no" active="yes"/>
+<layer number="25" name="tNames" color="7" fill="1" visible="yes" active="yes"/>
 <layer number="26" name="bNames" color="7" fill="1" visible="yes" active="yes"/>
-<layer number="27" name="tValues" color="7" fill="1" visible="no" active="yes"/>
+<layer number="27" name="tValues" color="7" fill="1" visible="yes" active="yes"/>
 <layer number="28" name="bValues" color="7" fill="1" visible="yes" active="yes"/>
 <layer number="29" name="tStop" color="7" fill="3" visible="no" active="yes"/>
@@
 </element>
 <element name="U$2" library="murata-dcdc" package="SMT" value="NTE0505SNTE0505MEC" x="22.5425" y="21.2725"/>
-<element name="C8" library="rcl" package="C0805" value="4,7µ" x="22.225" y="13.6525"/>
+<element name="C8" library="rcl" package="C0805" value="4,7µ" x="22.225" y="13.6525" rot="R180"/>
 <element name="R5" library="rcl" package="R0805" value="120" x="37.1475" y="6.6675" rot="R90"/>
 <element name="OK1" library="optocoupler" package="SMD8" value="6N137SMD-8" x="34.29" y="16.51" rot="R270"/>
@@
 <element name="R7" library="rcl" package="R0805" value="470" x="6.0325" y="6.35"/>
 <element name="R8" library="rcl" package="R0805" value="10k" x="32.385" y="24.13" rot="R180"/>
-<element name="R4" library="rcl" package="R0805" value="220" x="15.5575" y="11.1125" rot="R180"/>
-<element name="LED1" library="led" package="SML0603" value="" x="15.5575" y="13.0175"/>
+<element name="R4" library="rcl" package="R0805" value="220" x="14.605" y="12.7"/>
+<element name="LED1" library="led" package="SML0603" value="" x="18.415" y="13.335"/>
 <element name="R9" library="rcl" package="R0805" value="220" x="41.91" y="42.545" rot="R90"/>
 <element name="R10" library="rcl" package="R0805" value="220" x="41.91" y="38.4175" rot="R270"/>
@@
 </signal>
 <signal name="SVCC">
-<contactref element="U$2" pad="7"/>
 <contactref element="C6" pad="2"/>
 <contactref element="IC1" pad="8"/>
 <contactref element="IC2" pad="2"/>
 <contactref element="IC2" pad="3"/>
-<contactref element="C8" pad="1"/>
 <contactref element="IC2" pad="8"/>
 <contactref element="C5" pad="2"/>
-<wire x1="17.6925" y1="17.4625" x2="19.05" y2="17.4625" width="0.4064" layer="1"/>
-<wire x1="19.05" y1="17.4625" x2="21.2725" y2="15.24" width="0.4064" layer="1"/>
-<wire x1="21.2725" y1="15.24" x2="21.2725" y2="15.2425" width="0.4064" layer="1"/>
-<wire x1="21.2725" y1="15.2425" x2="21.275" y2="13.6525" width="0.4064" layer="1"/>
 <contactref element="OK1" pad="7"/>
 <wire x1="28.3591" y1="6.985" x2="28.3591" y2="5.715" width="0.4064" layer="1"/>
-<wire x1="21.275" y1="13.6525" x2="21.275" y2="15.2425" width="0.4064" layer="1"/>
-<contactref element="LED1" pad="A"/>
-<wire x1="21.275" y1="8.255" x2="21.275" y2="12.7" width="0.4064" layer="1"/>
-<wire x1="21.275" y1="12.7" x2="21.275" y2="13.6525" width="0.4064" layer="1"/>
-<wire x1="16.3075" y1="13.0175" x2="21.275" y2="13.0175" width="0.254" layer="1"/>
-<wire x1="21.275" y1="13.0175" x2="21.275" y2="12.7" width="0.254" layer="1"/>
 <wire x1="36.195" y1="12.0015" x2="35.56" y2="12.0015" width="0.4064" layer="1"/>
 <wire x1="35.875" y1="11.6865" x2="35.56" y2="12.0015" width="0.4064" layer="1"/>
@@
 <wire x1="25.4" y1="6.665" x2="25.4" y2="6.985" width="0.254" layer="1"/>
 <wire x1="36.195" y1="12.0015" x2="38.1" y2="12.0015" width="0.4064" layer="1"/>
+<contactref element="U$2" pad="8"/>
+<contactref element="C8" pad="2"/>
+<contactref element="LED1" pad="A"/>
+<wire x1="27.3925" y1="17.4625" x2="23.8125" y2="17.4625" width="0.4064" layer="1"/>
+<wire x1="23.8125" y1="17.4625" x2="21.2725" y2="14.9225" width="0.4064" layer="1"/>
+<wire x1="21.2725" y1="14.9225" x2="21.2725" y2="13.655" width="0.4064" layer="1"/>
+<wire x1="21.2725" y1="13.655" x2="21.275" y2="13.6525" width="0.4064" layer="1"/>
+<wire x1="21.275" y1="13.6525" x2="21.275" y2="8.255" width="0.4064" layer="1"/>
+<wire x1="21.275" y1="13.6525" x2="19.4825" y2="13.6525" width="0.254" layer="1"/>
+<wire x1="19.4825" y1="13.6525" x2="19.165" y2="13.335" width="0.254" layer="1"/>
 </signal>
 <signal name="SGND">
@@
 <contactref element="IC1" pad="2"/>
 <wire x1="10.2616" y1="3.81" x2="10.2616" y2="5.08" width="0.4064" layer="1"/>
-<contactref element="R4" pad="1"/>
-<contactref element="C8" pad="2"/>
-<contactref element="U$2" pad="8"/>
-<wire x1="27.3925" y1="17.4625" x2="25.4" y2="17.4625" width="0.4064" layer="1"/>
-<wire x1="25.4" y1="17.4625" x2="23.1775" y2="15.24" width="0.4064" layer="1"/>
-<wire x1="23.1775" y1="15.24" x2="23.1775" y2="13.655" width="0.4064" layer="1"/>
-<wire x1="23.1775" y1="13.655" x2="23.175" y2="13.6525" width="0.4064" layer="1"/>
-<wire x1="23.175" y1="13.6525" x2="23.175" y2="11.7475" width="0.4064" layer="1"/>
 <via x="19.05" y="11.745" extent="1-16" drill="0.7" shape="square"/>
 <via x="23.175" y="11.7475" extent="1-16" drill="0.7" shape="square"/>
@@
 <wire x1="19.05" y1="11.7475" x2="23.175" y2="11.7475" width="0.4064" layer="16"/>
 <wire x1="19.05" y1="11.745" x2="19.05" y2="11.7475" width="0.4064" layer="16"/>
-<wire x1="19.05" y1="11.745" x2="17.14" y2="11.745" width="0.4064" layer="1"/>
-<wire x1="17.14" y1="11.745" x2="16.5075" y2="11.1125" width="0.4064" layer="1"/>
 <wire x1="12.385" y1="8.255" x2="12.385" y2="8.575" width="0.4064" layer="1"/>
 <wire x1="12.385" y1="8.575" x2="13.335" y2="9.525" width="0.4064" layer="1"/>
-<wire x1="13.335" y1="9.525" x2="15.5575" y2="9.525" width="0.4064" layer="1"/>
-<wire x1="15.5575" y1="9.525" x2="16.51" y2="10.4775" width="0.4064" layer="1"/>
-<wire x1="16.51" y1="10.4775" x2="16.51" y2="11.11" width="0.4064" layer="1"/>
-<wire x1="16.51" y1="11.11" x2="16.5075" y2="11.1125" width="0.4064" layer="1"/>
+<wire x1="13.335" y1="9.525" x2="13.6525" y2="9.525" width="0.4064" layer="1"/>
+<wire x1="13.6525" y1="9.525" x2="15.5575" y2="9.525" width="0.4064" layer="1"/>
 <wire x1="12.385" y1="8.575" x2="8.57" y2="8.575" width="0.4064" layer="1"/>
 <wire x1="8.57" y1="8.575" x2="7.62" y2="9.525" width="0.4064" layer="1"/>
@@
 <wire x1="17.145" y1="1.27" x2="33.9725" y2="1.27" width="0.4064" layer="16"/>
 <wire x1="33.9725" y1="1.27" x2="36.5125" y2="3.81" width="0.4064" layer="16"/>
+<contactref element="R4" pad="1"/>
+<contactref element="C8" pad="1"/>
+<contactref element="U$2" pad="7"/>
+<wire x1="19.05" y1="11.745" x2="17.7775" y2="11.745" width="0.4064" layer="1"/>
+<wire x1="17.7775" y1="11.745" x2="15.5575" y2="9.525" width="0.4064" layer="1"/>
+<wire x1="13.655" y1="12.7" x2="13.655" y2="9.5275" width="0.4064" layer="1"/>
+<wire x1="13.655" y1="9.5275" x2="13.6525" y2="9.525" width="0.4064" layer="1"/>
+<wire x1="17.6925" y1="17.4625" x2="17.6925" y2="17.375" width="0.4064" layer="1"/>
+<wire x1="17.6925" y1="17.375" x2="13.6525" y2="13.335" width="0.4064" layer="1"/>
+<wire x1="13.6525" y1="13.335" x2="13.6525" y2="12.7025" width="0.4064" layer="1"/>
+<wire x1="13.6525" y1="12.7025" x2="13.655" y2="12.7" width="0.4064" layer="1"/>
 </signal>
 <signal name="N$20">
@@
 <contactref element="R4" pad="2"/>
 <contactref element="LED1" pad="C"/>
-<wire x1="14.6075" y1="11.1125" x2="14.8075" y2="11.3125" width="0.254" layer="1"/>
-<wire x1="14.8075" y1="11.3125" x2="14.8075" y2="13.0175" width="0.254" layer="1"/>
+<wire x1="17.665" y1="13.335" x2="16.19" y2="13.335" width="0.254" layer="1"/>
+<wire x1="16.19" y1="13.335" x2="15.555" y2="12.7" width="0.254" layer="1"/>
 </signal>
 <signal name="N$22">
